File: pcb/Converter_CN6009/Converter_CN6009.sch (KiCad schematic (older format))
At the start: 15 parts, among them J1 IN+, J2 IN-, J3 OUT+, J4 OUT-

Commit message: se realizo ruteo de pcb y correciones
Parts:
- removed D1: SS34, SS34:DIOM7959X265N, symbol SS34:SS34
- removed R1: 50K, Potentiometer_THT:Potentiometer_Bourns_3299W_Vertical, symbol Device:RTRIM
- added D1: SS34, Diode_SMD:D_SMA, symbol Device:D_Schottky
- added RV1: 50K, Potentiometer_THT:Potentiometer_Bourns_3296W_Vertical, symbol Device:R_POT_TRIM
- C2, C3: footprint Capacitor_SMD:C_0402_1005Metric -> Capacitor_SMD:C_0805_2012Metric
- L1: footprint Inductor_SMD:L_12x12mm_H8mm -> Inductor_SMD:L_Bourns_SRR1260
- R2: footprint Resistor_SMD:R_0603_1608Metric_Pad0.98x0.95mm_HandSolder -> Resistor_SMD:R_0805_2012Metric
- renumbered VR1 to U1
Connections:
- net at L1.2, U1.3 (SW): now also D1.2 (A)
- net at R2.1, U1.5 (FB): now also RV1.3
- net at C3.1, C4.1, J3.1 (Pin_1): now also D1.1 (K), RV1.1, RV1.2
Other:
- moved on the sheet: C3, C4, J3, J4
Changed lines of the file:
@@
 F 0 "C2" H 4465 3546 50  0000 L CNN
 F 1 "1uF" H 4465 3455 50  0000 L CNN
-F 2 "Capacitor_SMD:C_0402_1005Metric" H 4388 3350 50  0001 C CNN
+F 2 "Capacitor_SMD:C_0805_2012Metric" H 4388 3350 50  0001 C CNN
 F 3 "~" H 4350 3500 50  0001 C CNN
 	1    4350 3500
@@
 F 0 "L1" H 5450 2915 50  0000 C CNN
 F 1 "470uH" H 5450 2824 50  0000 C CNN
-F 2 "Inductor_SMD:L_12x12mm_H8mm" H 5450 2700 50  0001 C CNN
+F 2 "Inductor_SMD:L_Bourns_SRR1260" H 5450 2700 50  0001 C CNN
 F 3 "~" H 5450 2700 50  0001 C CNN
 	1    5450 2700
@@
 F 0 "R2" H 6970 3696 50  0000 L CNN
 F 1 "1.3K" H 6970 3605 50  0000 L CNN
-F 2 "Resistor_SMD:R_0603_1608Metric_Pad0.98x0.95mm_HandSolder" V 6830 3650 50  0001 C CNN
+F 2 "Resistor_SMD:R_0805_2012Metric" V 6830 3650 50  0001 C CNN
 F 3 "~" H 6900 3650 50  0001 C CNN
 	1    6900 3650
@@
 $EndComp
 $Comp
-L Device:RTRIM R1
-U 1 1 61104E3E
-P 6900 3050
-F 0 "R1" H 7028 3096 50  0000 L CNN
-F 1 "50K" H 7028 3005 50  0000 L CNN
-F 2 "Potentiometer_THT:Potentiometer_Bourns_3299W_Vertical" V 6830 3050 50  0001 C CNN
-F 3 "~" H 6900 3050 50  0001 C CNN
-	1    6900 3050
-	1    0    0    -1
-$EndComp
-$Comp
 L Device:CP1 C4
 U 1 1 611053B9
-P 7750 3500
-F 0 "C4" H 7865 3546 50  0000 L CNN
-F 1 "100uF" H 7865 3455 50  0000 L CNN
-F 2 "Capacitor_SMD:CP_Elec_8x10" H 7750 3500 50  0001 C CNN
-F 3 "~" H 7750 3500 50  0001 C CNN
-	1    7750 3500
+P 7850 3500
+F 0 "C4" H 7965 3546 50  0000 L CNN
+F 1 "100uF" H 7965 3455 50  0000 L CNN
+F 2 "Capacitor_SMD:CP_Elec_8x10" H 7850 3500 50  0001 C CNN
+F 3 "~" H 7850 3500 50  0001 C CNN
+	1    7850 3500
 	1    0    0    -1
 $EndComp
@@
 L Device:C C3
 U 1 1 61105DCA
-P 7300 3500
-F 0 "C3" H 7415 3546 50  0000 L CNN
-F 1 "1uF" H 7415 3455 50  0000 L CNN
-F 2 "Capacitor_SMD:C_0402_1005Metric" H 7338 3350 50  0001 C CNN
-F 3 "~" H 7300 3500 50  0001 C CNN
-	1    7300 3500
+P 7400 3500
+F 0 "C3" H 7515 3546 50  0000 L CNN
+F 1 "1uF" H 7515 3455 50  0000 L CNN
+F 2 "Capacitor_SMD:C_0805_2012Metric" H 7438 3350 50  0001 C CNN
+F 3 "~" H 7400 3500 50  0001 C CNN
+	1    7400 3500
 	1    0    0    -1
 $EndComp
@@
 L Connector:Conn_01x01_Female J3
 U 1 1 61106E5B
-P 8400 3150
-F 0 "J3" H 8500 3250 50  0000 L CNN
-F 1 "OUT+" H 8450 3150 50  0000 L CNN
-F 2 "Connector_Wire:SolderWire-0.75sqmm_1x01_D1.25mm_OD3.5mm" H 8400 3150 50  0001 C CNN
-F 3 "~" H 8400 3150 50  0001 C CNN
-	1    8400 3150
+P 8500 3150
+F 0 "J3" H 8600 3250 50  0000 L CNN
+F 1 "OUT+" H 8550 3150 50  0000 L CNN
+F 2 "Connector_Wire:SolderWire-0.75sqmm_1x01_D1.25mm_OD3.5mm" H 8500 3150 50  0001 C CNN
+F 3 "~" H 8500 3150 50  0001 C CNN
+	1    8500 3150
 	1    0    0    -1
 $EndComp
@@
 L Connector:Conn_01x01_Female J4
 U 1 1 61107569
-P 8450 3950
-F 0 "J4" H 8550 4050 50  0000 L CNN
-F 1 "OUT-" H 8500 3950 50  0000 L CNN
-F 2 "Connector_Wire:SolderWire-0.75sqmm_1x01_D1.25mm_OD3.5mm" H 8450 3950 50  0001 C CNN
-F 3 "~" H 8450 3950 50  0001 C CNN
-	1    8450 3950
+P 8550 3950
+F 0 "J4" H 8650 4050 50  0000 L CNN
+F 1 "OUT-" H 8600 3950 50  0000 L CNN
+F 2 "Connector_Wire:SolderWire-0.75sqmm_1x01_D1.25mm_OD3.5mm" H 8550 3950 50  0001 C CNN
+F 3 "~" H 8550 3950 50  0001 C CNN
+	1    8550 3950
 	1    0    0    -1
 $EndComp
@@
 Wire Wire Line
 	6050 3950 4350 3950
-$Comp
-L SS34:SS34 D1
-U 1 1 61134CE2
-P 6450 2700
-F 0 "D1" H 6450 2917 50  0000 C CNN
-F 1 "SS34" H 6450 2826 50  0000 C CNN
-F 2 "SS34:DIOM7959X265N" H 6450 2700 50  0001 C CNN
-F 3 "DO-214 ON Semiconductor" H 6450 2700 50  0001 L BNN
-F 4 "SS Series 500 mV 3 A 40 V Max Reverse Voltage Schottky Rectifier - DO-214AB" H 6450 2700 50  0001 L BNN "Field4"
-F 5 "None" H 6450 2700 50  0001 L BNN "Field5"
-F 6 "SS34" H 6450 2700 50  0001 L BNN "Field6"
-F 7 "Unavailable" H 6450 2700 50  0001 L BNN "Field7"
-F 8 "ON Semiconductor" H 6450 2700 50  0001 L BNN "Field8"
-	1    6450 2700
-	1    0    0    -1
-$EndComp
 Connection ~ 6050 3950
 Wire Wire Line
-	8250 3950 7750 3950
-Wire Wire Line
-	7300 3650 7300 3950
-Connection ~ 7300 3950
-Wire Wire Line
-	7750 3650 7750 3950
-Connection ~ 7750 3950
-Wire Wire Line
-	7750 3950 7300 3950
+	8350 3950 7850 3950
+Wire Wire Line
+	7850 3650 7850 3950
+Connection ~ 7850 3950
 $Comp
 L power:GND #PWR0101
 U 1 1 61161E7F
-P 6050 4100
-F 0 "#PWR0101" H 6050 3850 50  0001 C CNN
-F 1 "GND" H 6055 3927 50  0000 C CNN
-F 2 "" H 6050 4100 50  0001 C CNN
-F 3 "" H 6050 4100 50  0001 C CNN
-	1    6050 4100
-	1    0    0    -1
-$EndComp
-Wire Wire Line
-	6050 4100 6050 3950
+P 3850 4100
+F 0 "#PWR0101" H 3850 3850 50  0001 C CNN
+F 1 "GND" H 3855 3927 50  0000 C CNN
+F 2 "" H 3850 4100 50  0001 C CNN
+F 3 "" H 3850 4100 50  0001 C CNN
+	1    3850 4100
+	1    0    0    -1
+$EndComp
 $Comp
 L power:PWR_FLAG #FLG0101
@@
 $EndComp
 $Comp
-L XL6009:XL6009 VR1
+L XL6009:XL6009 U1
 U 1 1 6115EEA5
 P 5450 3350
-F 0 "VR1" H 5450 3817 50  0000 C CNN
+F 0 "U1" H 5450 3817 50  0000 C CNN
 F 1 "XL6009" H 5450 3726 50  0000 C CNN
 F 2 "XL6009:DPAK170P1435X465-6N" H 5450 3350 50  0001 L BNN
@@
 Text Notes 3000 3550 0    79   ~ 0
 Vin
-Text Notes 8350 3550 0    79   ~ 0
+Text Notes 8450 3550 0    79   ~ 0
 Vout
-Wire Wire Line
-	6050 3950 6900 3950
-Wire Wire Line
-	6900 3800 6900 3950
-Connection ~ 6900 3950
-Wire Wire Line
-	6900 3950 7300 3950
 Wire Wire Line
 	5950 3350 6900 3350
@@
 	3000 4900 3000 5750
 Wire Wire Line
-	6900 3200 6900 3350
-Connection ~ 6900 3350
-Wire Wire Line
 	5700 2700 6050 2700
 Wire Wire Line
@@
 	4800 2700 4800 3150
 Wire Wire Line
-	8200 3150 8100 3150
-Wire Wire Line
-	8100 3150 8100 2700
-Wire Wire Line
-	8100 2700 7750 2700
-Wire Wire Line
-	6900 2900 6900 2700
-Connection ~ 6900 2700
-Wire Wire Line
-	6900 2700 6550 2700
-Wire Wire Line
-	7300 3350 7300 2700
-Connection ~ 7300 2700
-Wire Wire Line
-	7300 2700 6900 2700
-Wire Wire Line
-	7750 3350 7750 2700
-Connection ~ 7750 2700
-Wire Wire Line
-	7750 2700 7300 2700
+	8300 3150 8200 3150
+Wire Wire Line
+	8200 3150 8200 2700
+Wire Wire Line
+	8200 2700 7850 2700
+Wire Wire Line
+	7400 3350 7400 2700
+Wire Wire Line
+	7850 3350 7850 2700
+Connection ~ 7850 2700
+Wire Wire Line
+	7850 2700 7400 2700
 Wire Wire Line
 	5950 3150 6050 3150
 Wire Wire Line
 	6050 3150 6050 2700
-Connection ~ 6050 2700
-Wire Wire Line
-	6050 2700 6350 2700
-Text Notes 3900 2250 0    91   ~ 0
+Text Notes 3900 2200 0    91   ~ 0
 XL6009 Typical Application Circuit (Boost Converter)
-Text Notes 8750 3300 0    59   ~ 0
+Text Notes 8850 3300 0    59   ~ 0
 Voltaje de salida
 Text Notes 2000 3300 0    59   ~ 0
 Voltaje de entrada
 Wire Notes Line
-	8650 3550 8750 3350
-Wire Notes Line
-	8750 3350 9550 3350
+	8750 3550 8850 3350
+Wire Notes Line
+	8850 3350 9650 3350
 Wire Notes Line
 	2950 3550 2850 3350
 Wire Notes Line
 	2850 3350 2000 3350
+Wire Wire Line
+	3850 4100 3850 3950
+$Comp
+L power:GND #PWR0102
+U 1 1 61200243
+P 7850 4100
+F 0 "#PWR0102" H 7850 3850 50  0001 C CNN
+F 1 "GND" H 7855 3927 50  0000 C CNN
+F 2 "" H 7850 4100 50  0001 C CNN
+F 3 "" H 7850 4100 50  0001 C CNN
+	1    7850 4100
+	1    0    0    -1
+$EndComp
+Wire Wire Line
+	7850 4100 7850 3950
+$Comp
+L power:GND #PWR0103
+U 1 1 61202535
+P 6050 4100
+F 0 "#PWR0103" H 6050 3850 50  0001 C CNN
+F 1 "GND" H 6055 3927 50  0000 C CNN
+F 2 "" H 6050 4100 50  0001 C CNN
+F 3 "" H 6050 4100 50  0001 C CNN
+	1    6050 4100
+	1    0    0    -1
+$EndComp
+Wire Wire Line
+	6050 4100 6050 3950
+$Comp
+L Device:D_Schottky D1
+U 1 1 61203570
+P 6450 2700
+F 0 "D1" H 6450 2483 50  0000 C CNN
+F 1 "SS34" H 6450 2574 50  0000 C CNN
+F 2 "Diode_SMD:D_SMA" H 6450 2700 50  0001 C CNN
+F 3 "~" H 6450 2700 50  0001 C CNN
+	1    6450 2700
+	-1   0    0    1
+$EndComp
+Wire Wire Line
+	6300 2700 6050 2700
+Connection ~ 6050 2700
+$Comp
+L Device:R_POT_TRIM RV1
+U 1 1 6121650C
+P 6900 3000
+F 0 "RV1" H 7100 2900 50  0000 R CNN
+F 1 "50K" H 7100 2800 50  0000 R CNN
+F 2 "Potentiometer_THT:Potentiometer_Bourns_3296W_Vertical" H 6900 3000 50  0001 C CNN
+F 3 "~" H 6900 3000 50  0001 C CNN
+	1    6900 3000
+	1    0    0    -1
+$EndComp
+Wire Wire Line
+	6900 3150 6900 3350
+Connection ~ 6900 3350
+Wire Wire Line
+	6900 2850 6900 2800
+Wire Wire Line
+	7050 3000 7100 3000
+Wire Wire Line
+	7100 3000 7100 2800
+Wire Wire Line
+	7100 2800 6900 2800
+Connection ~ 6900 2800
+Wire Wire Line
+	6900 2800 6900 2700
+Wire Wire Line
+	6900 3800 6900 3950
+Wire Wire Line
+	7400 3650 7400 3950
+Wire Wire Line
+	7400 3950 7850 3950
+Wire Wire Line
+	6600 2700 6900 2700
+Wire Wire Line
+	6050 3950 6900 3950
+Wire Wire Line
+	6900 2700 7400 2700
+Connection ~ 6900 2700
+Connection ~ 7400 2700
+Wire Wire Line
+	6900 3950 7400 3950
+Connection ~ 6900 3950
+Connection ~ 7400 3950
 $EndSCHEMATC

Commit message: se realizo todas las correcciones para la revision final
Parts:
- added FID1: Fiducial, Fiducial:Fiducial_0.75mm_Mask1.5mm, symbol Mechanical:Fiducial
- IN+1: renamed from J1; value IN+ -> J1
- IN-1: renamed from J2; value IN- -> J2
- OUT+1: renamed from J3; value OUT+ -> J3
- OUT-1: renamed from J4; value OUT- -> J4
Other:
- note added: "Fiducial"
- moved on the sheet: H1, H2
